File: hardware/design/watch_design_v2.kicad_sch (KiCad schematic)
At the start: 63 parts, among them J1 BAT, J2 USB_C_Receptacle_USB2.0, J3 SWDIO, J4 SWDCLK, J5 ~{RST}, J6 SWO, J7 GND, Q1 BSS138, SW1 SW_Push, SW2 SW_Push, U1 MAX86141ENP+T, U2 SFH_7015, U3 RV-8523-C3, U4 LSM6DSOXTR, U5 NPM1300-QEAA-R7, U6 NINA-B306-00B-00, U7 GC9A01_IPS_display_SPI, U8 LIS2DS12, U9 MAX32664GTGC_

Commit message: updated design files with appropriate parts
Parts:
- removed LED2: CT DBLP31.12-6C5D-56-J6Q4, FIREFLY E2218:CT DBLP31.12-6C5D-56-J6Q4_OSR, symbol FIREFLY E2218:CT_DBLP31.12-6C5D-56-J6Q4
- removed U3: RV-8523-C3, Package_SON:RTC_SMD_MicroCrystal_C3_2.5x3.7mm, symbol Timer_RTC:RV-8523-C3
- removed U6: NINA-B306-00B-00, NINA-B306-00B-00:XCVR_NINA-B306-00B-00, symbol NINA-B306:NINA-B306-00B-00
- added LED4: CT DBLP31.12-6C5D-56-J6Q4, CT DBLP31.12-6C5D-56-J6Q4_OSR, symbol FIREFLY E2218:CT_DBLP31.12-6C5D-56-J6Q4
- added U3: RV-8263-C8 32.768KHZ 20PPM TA QA, easyeda2kicad:OSC-SMD_8P-L2.0-W1.2, symbol rv8263-c8:RV-8263-C832.768KHZ20PPMTAQA
- added U6: NINA-B306-00B-00, XCVR_NINA-B306-00B-00, symbol NINA-B306-00B-00:NINA-B306-00B-00
- LED1, LED3: footprint SFH-2703:SFH2703 -> SFH2703
- U1: footprint MAX86141:BGA-20_L2.0-W1.8-R4-C5-P0.40-TL -> easyeda2kicad:BGA-20_L2.0-W1.8-R4-C5-P0.40-TL
- U2: value SFH_7015 -> SFH 7015; footprint SFH-7015:SFH 7015_OSR -> SFH 7015_OSR
- U4: footprint LSM6DSOXTR:PQFN50P250X300X86-14N -> PQFN50P250X300X86-14N; LCSC Part C481766 -> (none)
- U5: footprint npm1300_qfn:QFN-32_L5.0-W5.0-P0.50-TL-EP3.5 -> easyeda2kicad:QFN-32_L5.0-W5.0-P0.50-TL-EP3.5
- U8: footprint LIS2DS12:LGA-12_L2.0-W2.0-P0.50-BL -> easyeda2kicad:LGA-12_L2.0-W2.0-P0.50-BL
- U9: LCSC Part C5344734 -> (none)
Connections:
- net +1V8: now also U3.5 (VDD), U6.10 (VCC), U6.9 (VCC_IO); no longer U9.22 (VDD__1)
- net BTN1: now also U6.4 (GPIO_4)
- net D+: now also U6.54 (USB_DP)
- net D-: now also U6.55 (USB_DM)
- net GND: now also U3.4 (VSS), U6.12 (GND), U6.14 (GND), U6.26 (GND), U6.30 (GND), U6.53 (GND), U6.6 (GND), U6.EAGP1 (EAGP), U6.EAGP2 (EAGP), U6.EAGP3 (EAGP), U6.EAGP4 (EAGP), U6.EGP1 (EGP), U6.EGP10 (EGP), U6.EGP11 (EGP), U6.EGP12 (EGP), U6.EGP2 (EGP), U6.EGP3 (EGP), U6.EGP4 (EGP), U6.EGP5 (EGP), U6.EGP6 (EGP), U6.EGP7 (EGP), U6.EGP8 (EGP), U6.EGP9 (EGP); no longer U8.5 (NC)
- net GREEN: now also LED4.1, LED4.3
- net MEM_INT1: now also U6.17 (GPIO_17)
- net MEM_INT2: now also U6.18 (GPIO_18)
- net MFIO: now also U6.5 (GPIO_5)
- net SCL: now also U3.8 (SCL), U6.48 (QSPI_D1/GPIO_48)
- net SDA: now also U3.1 (SDA), U6.49 (QSPI_D2/GPIO_49)
- net SHPHLD: now also U6.47 (QSPI_D3/GPIO_47)
- net SQW: now also U3.7 (CLKOUT)
- net SWDCLK: now also U6.11 (SWDCLK)
- net SWDIO: now also U6.15 (SWDIO)
- net SWO: now also U6.8 (SWO/TRACE_D0/GPIO_8)
- net TFT_BCKL: now also U6.3 (GPIO_3)
- net TFT_DC: now also U6.24 (GPIO_24)
- net TFT_MOSI: now also U6.21 (GPIO_21)
- net TFT_SCK: now also U6.22 (GPIO_22)
- net VBUS: now also U6.31 (VBUS)
- net VCC: now also LED4.2
- net ~{MAX_RST}: now also U6.7 (GPIO_7)
- net ~{RST}: now also U6.19 (~{RESET})
- net ~{TFT_CS}: now also U6.23 (GPIO_23)
- new net CLKOE: U3.2 (CLKOE), U6.20 (GPIO_20)
- no-connect marks 53 -> 54
Other:
- note removed: "change this to rv8263-c8"
- moved on the sheet: C4

Commit message: restructured files
Parts:
- removed R11: 4.7k, Resistor_SMD:R_0603_1608Metric, symbol Device:R
- removed R7: 1k, Resistor_SMD:R_0603_1608Metric, symbol Device:R_Small
- removed R8: 100n, Resistor_SMD:R_0603_1608Metric, symbol Device:R_Small
- added R2: 47k, Resistor_SMD:R_0603_1608Metric, symbol Device:R_Small
- added R3: 100, Resistor_SMD:R_0603_1608Metric, symbol Device:R_Small
- LED1, LED3: footprint SFH2703 -> SFH-2703:SFH2703
- LED4: footprint CT DBLP31.12-6C5D-56-J6Q4_OSR -> FIREFLY E2218:CT DBLP31.12-6C5D-56-J6Q4_OSR
- R1: value 47k -> 1k
- SW1, SW2: footprint LXTD-0204-034:SW-SMD_LXTD-0204-034 -> OSW:button_side_smd
- U1: footprint easyeda2kicad:BGA-20_L2.0-W1.8-R4-C5-P0.40-TL -> MAX86141:BGA-20_L2.0-W1.8-R4-C5-P0.40-TL
- U2: footprint SFH 7015_OSR -> SFH-7015:SFH7015
- U3: footprint easyeda2kicad:OSC-SMD_8P-L2.0-W1.2 -> rv8263-c8:OSC-SMD_8P-L2.0-W1.2
- U4: footprint PQFN50P250X300X86-14N -> LSM6DSOXTR:PQFN50P250X300X86-14N
- U5: footprint easyeda2kicad:QFN-32_L5.0-W5.0-P0.50-TL-EP3.5 -> npm1300_qfn:QFN-32_L5.0-W5.0-P0.50-TL-EP3.5
- U6: footprint XCVR_NINA-B306-00B-00 -> NINA-B306-00B-00:XCVR_NINA-B306-00B-00
- U8: footprint easyeda2kicad:LGA-12_L2.0-W2.0-P0.50-BL -> LIS2DS12:LGA-12_L2.0-W2.0-P0.50-BL
Connections:
- net +1V8: now also R1.1, U9.22 (VDD__1)
- net +BATT: now also J1.2 (Pin_2); no longer J1.1 (Pin_1)
- net BTN1: now also R1.2
- net GND: now also J1.1 (Pin_1), R2.2; no longer J1.2 (Pin_2), R1.2
- net SQW: no longer R6.2
- net VSET1: now also R2.1; no longer R1.1
- net VUSB: no longer C6.1, U5.21 (VBUS)
- net ~{MAX_RST_0}: now also R3.2
- net ~{MAX_RST}: now also R3.1
- net ~{PPG_INT}: now also R6.2
- new net VDD: C6.1, U5.21 (VBUS)
Other:
- moved on the sheet: C10, C8

Commit message: updated design as a two part pcb
Parts:
- removed C1, C15, C18, C19, C20, C21, C6: 1u, Capacitor_SMD:C_0603_1608Metric, symbol Device:C_Small
- removed C10, C14, C2, C24, C25, C4, C7, C8: 100n, Capacitor_SMD:C_0603_1608Metric, symbol Device:C_Small
- removed C11, C12: 100n, Capacitor_SMD:C_0603_1608Metric, symbol Device:C
- removed C13, C22, C3, C5: 10u, Capacitor_SMD:C_0603_1608Metric, symbol Device:C_Small
- removed C9: 2.2u, Capacitor_SMD:C_0603_1608Metric, symbol Device:C_Small
- removed J1: BAT, Connector_JST:JST_ACH_BM02B-ACHSS-GAN-ETF_1x02-1MP_P1.20mm_Vertical, symbol Connector_Generic:Conn_01x02
- removed J2: USB_C_Receptacle_USB2.0, Connector_USB:USB_C_Receptacle_GCT_USB4110, symbol Connector:USB_C_Receptacle_USB2.0
- removed J3: SWDIO, Connector_Wire:SolderWirePad_1x01_SMD_1x2mm, symbol Connector_Generic:Conn_01x01
- removed J4: SWDCLK, Connector_Wire:SolderWirePad_1x01_SMD_1x2mm, symbol Connector_Generic:Conn_01x01
- removed J5: ~{RST}, Connector_Wire:SolderWirePad_1x01_SMD_1x2mm, symbol Connector_Generic:Conn_01x01
- removed J6: SWO, Connector_Wire:SolderWirePad_1x01_SMD_1x2mm, symbol Connector_Generic:Conn_01x01
- removed J7: GND, Connector_Wire:SolderWirePad_1x01_SMD_1x2mm, symbol Connector_Generic:Conn_01x01
- removed JP1: SolderJumper_2_Open, Jumper:SolderJumper-2_P1.3mm_Open_RoundedPad1.0x1.5mm, symbol Jumper:SolderJumper_2_Open
- removed L1: 2.2uH, Inductor_SMD:L_0603_1608Metric, symbol Device:L_Small
- removed LED1, LED3: SFH_2703, SFH-2703:SFH2703, symbol SFH_2703:SFH_2703
- removed LED4: CT DBLP31.12-6C5D-56-J6Q4, FIREFLY E2218:CT DBLP31.12-6C5D-56-J6Q4_OSR, symbol FIREFLY E2218:CT_DBLP31.12-6C5D-56-J6Q4
- removed Q1: BSS138, Package_TO_SOT_SMD:SOT-23, symbol Transistor_FET:BSS138
- removed R1: 1k, Resistor_SMD:R_0603_1608Metric, symbol Device:R_Small
- removed R10: 470, Resistor_SMD:R_0603_1608Metric, symbol Device:R
- removed R2: 47k, Resistor_SMD:R_0603_1608Metric, symbol Device:R_Small
- removed R3: 100, Resistor_SMD:R_0603_1608Metric, symbol Device:R_Small
- removed R4, R5, R6: 4.7k, Resistor_SMD:R_0603_1608Metric, symbol Device:R
- removed R9: 47k, Resistor_SMD:R_0603_1608Metric, symbol Device:R
- removed SW1, SW2: SW_Push, OSW:button_side_smd, symbol Switch:SW_Push
- removed TP1, TP2, TP3, TP4, TP5, TP6, TP7, TP8: TestPoint, TestPoint:TestPoint_Pad_D1.0mm, symbol Connector:TestPoint
- removed U1: MAX86141ENP+T, MAX86141:BGA-20_L2.0-W1.8-R4-C5-P0.40-TL, symbol MAX86141:MAX86141ENP+T
- removed U2: SFH 7015, SFH-7015:SFH7015, symbol SFH-7015:SFH_7015
- removed U3: RV-8263-C8 32.768KHZ 20PPM TA QA, rv8263-c8:OSC-SMD_8P-L2.0-W1.2, symbol rv8263-c8:RV-8263-C832.768KHZ20PPMTAQA
- removed U4: LSM6DSOXTR, LSM6DSOXTR:PQFN50P250X300X86-14N, symbol LSM6DSOXTR:LSM6DSOXTR
- removed U5: NPM1300-QEAA-R7, npm1300_qfn:QFN-32_L5.0-W5.0-P0.50-TL-EP3.5, symbol npm1300_qfn:NPM1300-QEAA-R7
- removed U6: NINA-B306-00B-00, NINA-B306-00B-00:XCVR_NINA-B306-00B-00, symbol NINA-B306-00B-00:NINA-B306-00B-00
- removed U7: GC9A01_IPS_display_SPI, gc9a01_fpc:15p_tft_P0.5, symbol open_smartwatch:GC9A01_IPS_display_SPI
- removed U8: LIS2DS12, LIS2DS12:LGA-12_L2.0-W2.0-P0.50-BL, symbol LIS2DS12:LIS2DS12
- removed U9: MAX32664GTGC_, MAX32664GTGC_:IC_MAX32664GTGC_, symbol MAX32664GTGC_:MAX32664GTGC_
Connections:
- no-connect marks 54 -> 0
Other:
- added sheet PPG (ppg.kicad_sch)
- added sheet main_board (main_board.kicad_sch)
- note removed: "3.3v-5v ~31.2mA"
- note removed: "6D IMU"
- note removed: "BOOTLOADER MODE: 1. Set rstn pin low for 10ms 2. while rstn pin is low, set mfio low 3. After 10s set rstn pin high 4. After additional 50ms, bootloader mode entered APPLICATION MODE: 1. Set rstn pin low for 10ms 2. while rstn pin is low, set mfio high 3. After 10s, set rstn pin high 4. After additional 50ms, application mode entered"
- note removed: "Blood oxygen levels measured using red and IR light"
- note removed: "DISPLAY"
- note removed: "FLAGS"
- note removed: "HEART RATE AND PULSE OXIMETER"
- note removed: "I2C addr: 0x55"
- note removed: "I2C addr: 0x6A"
- note removed: "I2C addr: 0x6B"
- note removed: "NAVIGATORS"
- note removed: "NINA-B306 MCU"
- note removed: "POWER"
- note removed: "PULL UPS"
- note removed: "RTCC"
- note removed: "TEST POINTS"
- note removed: "This accelerometer is used for distance/motion artifact compensation in HRM and SpO2 tasks"
- note removed: "USB_C"
- note removed: "Vsys voltage is the same as Vbus voltage and is unregulated. VSET1 sets the output voltage of BUCK1 All other settings will be done via TWI"
- note removed: "buck converter + battery charger + fuel gauge"
- note removed: "consider 1.nina-w106 2.nora-w101/w106"
- note removed: "i2c addr: 0x68"
- note removed: "program using SPI interface. TFT_RST is an optional pin"
- note removed: "using an FPC connected with 15 lines and and pitch 0.5mm"
- note removed: "utilizing tap and double tap gestures for select and back gestures"
- note removed: "~{RST} & MFIO pin states cause sensor to enter either bootloader or application mode"
