File: hardware/design/main_board.kicad_sch (KiCad schematic)
At the start: 63 parts, among them J1 BAT, J2 USB_C_Receptacle_USB2.0, J3 SWDIO, J4 SWDCLK, J5 ~{RST}, J6 SWO, J7 GND, J9 HRM_F, SW1 SW_Push, SW2 SW_Push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

Commit message: updated design to include two boards connected back to back
Parts:
- added C23, C26: 100n, Capacitor_SMD:C_0603_1608Metric, symbol Device:C_Small
- SW1, SW2: footprint OSW:button_side_smd -> Button_Switch_SMD:SW_SPST_B3U-3000P-B
Connections:
- net +3.3V is gone; now on net +3V0: C17.1, L2.1
- net +3V0: now also C13.1
- net D+: now also D1.2 (I/O1); no longer D1.3 (I/O2)
- net D-: now also D1.3 (I/O2); no longer D1.2 (I/O1)
- net GND: now also C23.2, C26.2
- net SCL: now also U6.49 (QSPI_D2/GPIO_49); no longer U6.48 (QSPI_D1/GPIO_48)
- net SDA: now also U6.48 (QSPI_D1/GPIO_48); no longer U6.49 (QSPI_D2/GPIO_49)
- net TFT_DC: now also U6.21 (GPIO_21); no longer U6.24 (GPIO_24)
- net TFT_MOSI: now also U6.24 (GPIO_24); no longer U6.21 (GPIO_21)
- net TFT_SCK: now also U6.23 (GPIO_23); no longer U6.22 (GPIO_22)
- net VBUS: now also C23.1, C26.1
- net VCC: no longer C13.1
- net ~{TFT_CS}: now also U6.22 (GPIO_22); no longer U6.23 (GPIO_23)
- net ISET: now reaches R7.2, U10.5 (ISET)
- net SW2: now reaches L2.2, U5.5 (SW2)
