File: hardware/watch/watch.kicad_pcb (KiCad board)
At the start: 4 copper layers, 40 x 42.4 mm, 69 parts, among them J1 BAT, J2 USB_C_Receptacle_USB2.0, J3 SWDIO, J4 SWDCLK, J6 SWO, J7 GND, J9 HRM_F, SW1 SW_Push, SW2 SW_Push, U1 MAX86141ENP+T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

Commit message: updated designs
Parts:
- added TP11: TestPoint, TestPoint:TestPoint_Pad_D1.0mm, B.Cu at (145.3, 118.5)
- added kibuzzard-6A08DFE9: G***, kibuzzard-6A08DFE9, B.Cu at (166.3, 90.9)
- added kibuzzard-6A08DFFD: G***, kibuzzard-6A08DFFD, B.Cu at (166.8, 104.2)
- added kibuzzard-6A08E019: G***, kibuzzard-6A08E019, B.Cu at (152.6, 96.1)
- added kibuzzard-6A08E02E: G***, kibuzzard-6A08E02E, B.Cu at (156.2, 94.6)
- added kibuzzard-6A08E080: G***, kibuzzard-6A08E080, B.Cu at (142.2, 100.7)
- added kibuzzard-6A08E0DD: G***, kibuzzard-6A08E0DD, B.Cu at (147.3, 91.6)
- added kibuzzard-6A08E0EE: G***, kibuzzard-6A08E0EE, B.Cu at (149.9, 91.6)
- added kibuzzard-6A08E121: G***, kibuzzard-6A08E121, B.Cu at (134.7, 106.6)
- added kibuzzard-6A0A1465: G***, kibuzzard-6A0A1465, B.Cu at (156.7, 101.5)
- added kibuzzard-6A0A16D4: G***, kibuzzard-6A0A16D4, B.Cu at (143.2, 117.5)
- D1, TP9: moved to F.Cu
- TP5: moved to B.Cu
- moved TP10 26.9 mm to (154.1, 101.5)
- moved R7 19.3 mm to (143.5, 104.4), turned to 0 degrees
- moved C16 13.3 mm to (141.7, 108.0)
- moved U10 13.3 mm to (145.2, 107.8)
- moved TP6 10.9 mm to (164.5, 104.2)
- moved C25 10.1 mm to (162.7, 109.5)
- moved C24 10.1 mm to (165.1, 110.2)
- moved U11 10.1 mm to (165.1, 107.9)
- moved U3 8.47 mm to (164.2, 102.8), turned to 180 degrees
- moved TP5 8.21 mm to (166.3, 93.2), turned to 180 degrees
- moved TP9 8.09 mm to (151.2, 104.6), turned to 0 degrees
- moved C1 7.67 mm to (153.8, 108.5)
- moved C18 7.67 mm to (157.8, 107.7)
- moved C19 7.67 mm to (156.2, 107.7)
- moved C20 7.67 mm to (157.2, 100.3)
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Connections:
- U6 pad 1: SHPHLD -> MEM_INT2
- U6 pad 17: MEM_INT1 -> unconnected-(U6-GPIO_17-Pad17)
- U6 pad 18: MEM_INT2 -> unconnected-(U6-GPIO_18-Pad18)
- U6 pad 2: unconnected-(U6-GPIO_2-Pad2) -> MEM_INT1
- U6 pad 20: CLKOE -> unconnected-(U6-GPIO_20-Pad20)
- U6 pad 25: unconnected-(U6-GPIO_25-Pad25) -> TFT_BCKL
- U6 pad 3: TFT_BCKL -> CLKOE
Routing:
- net +1V8: track 2.01 -> 43.8 mm, vias 0 -> 14
- net SDA: track 22.4 -> 60.4 mm, vias 0 -> 1
- net GND: track 46.3 -> 82.1 mm, vias 61 -> 59
- net SCL: track 24.9 -> 59.8 mm, vias 1 -> 5
- net CLKOE: track 1.73 -> 20.3 mm, vias 1 -> 2
- net VCC: track 4.46 -> 20.2 mm, vias 0 -> 2
- net MEM_INT1: track 3.27 -> 17.6 mm
- net ~{PPG_INT}: track 15.1 -> 27.5 mm, vias 2 -> 3
- net /LEDK: track 14.8 -> 3.25 mm
- net ~{ACCEL_CS}: track 6.56 -> 17.7 mm
- net TFT_MOSI: track 36.1 -> 26.3 mm, vias 3 -> 1
- net TFT_SCK: track 36.9 -> 27.6 mm, vias 3 -> 2
- net PPG_CS: track 27.0 -> 18.0 mm
- net +3V0: track 15.7 -> 24.5 mm, vias 7 -> 6
- net MEM_INT2: track 5.84 -> 14.5 mm
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- added copper zone on In2.Cu, net +1V8
- added copper zone on In1.Cu, net GND
- removed copper zone on F.Cu, net +1V8
- removed copper zone on B.Cu, net GND
Other:
- outline, holes or cut-outs redrawn
- board text added: "bridge for tft_rst->rst"
