File: hardware/watch/watch.kicad_sch (KiCad schematic)
At the start: 70 parts, among them J1 BAT, J2 USB_C_Receptacle_USB2.0, J3 SWDIO, J4 SWDCLK, J5 ~{RST}, J6 SWO, J7 GND, J9 HRM_F, SW1 SW_Push, SW2 SW_Push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

Commit message: updated designs
Parts:
- added TP11: TestPoint, TestPoint:TestPoint_Pad_D1.0mm, symbol Connector:TestPoint
Connections:
- net +3V0: now also TP11.1
- net CLKOE: now also U6.3 (GPIO_3); no longer U6.20 (GPIO_20)
- net MEM_INT1: now also U6.2 (GPIO_2); no longer U6.17 (GPIO_17)
- net MEM_INT2: now also U6.1 (GPIO_1); no longer U6.18 (GPIO_18)
- net SHPHLD: no longer U6.1 (GPIO_1)
- net TFT_BCKL: now also U6.25 (GPIO_25); no longer U6.3 (GPIO_3)
- no-connect marks 57 -> 58
